File: hardware/quietbot.sch (EAGLE design)
At the start: 9 parts, among them IC2 REG1117

Commit message: board design
Parts:
- added J1: (no value), SparkFun-Connectors:M031X03_NO_SILK
- added J2: (no value), SparkFun-Connectors:M04NO_SILK_ALL_ROUND
- added R1, R6: 10K, resistor:R-EU_R0805
- added TP1: TPTP15R, testpad:TPTP15R
Connections:
- new net N$4: R6.2, TP1.TP, U$1.GPIO0
- new net N$5: R1.2, U$1.CH_PD
- new net RX: J2.2, U$1.RX
- new net SIG_PIXEL: J1.2, U$1.GPIO2
- new net TX: J2.3, U$1.TX
- net +3V3: now also J2.1, R1.1, R6.1; no longer U$1.CH_PD
- net +5V: now also J1.1
- net GND: now also J1.3, J2.4
Changed lines of the file:
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@@
 <part name="GND1" library="supply1" deviceset="GND" device=""/>
 <part name="GND3" library="supply1" deviceset="GND" device=""/>
-<part name="GND4" library="supply1" deviceset="GND" device=""/>
-<part name="GND5" library="supply1" deviceset="GND" device=""/>
 <part name="GND6" library="supply1" deviceset="GND" device=""/>
 <part name="U$2" library="rainsun-ant" deviceset="ANT" device=""/>
 <part name="+3V1" library="supply1" deviceset="+3V3" device=""/>
-<part name="+3V2" library="supply1" deviceset="+3V3" device=""/>
 <part name="+3V3" library="supply1" deviceset="+3V3" device=""/>
-<part name="+3V5" library="supply1" deviceset="+3V3" device=""/>
-<part name="GND7" library="supply1" deviceset="GND" device=""/>
-<part name="GND8" library="supply1" deviceset="GND" device=""/>
 <part name="GND9" library="supply1" deviceset="GND" device=""/>
-<part name="GND10" library="supply1" deviceset="GND" device=""/>
 <part name="R2" library="resistor" deviceset="R-EU_" device="R0805" value="1K"/>
 <part name="GND11" library="supply1" deviceset="GND" device=""/>
@@
 <part name="GND12" library="supply1" deviceset="GND" device=""/>
 <part name="R3" library="resistor" deviceset="R-EU_" device="R0805" value="10K"/>
+<part name="R6" library="resistor" deviceset="R-EU_" device="R0805" value="10K"/>
+<part name="+3V7" library="supply1" deviceset="+3V3" device=""/>
+<part name="TP1" library="testpad" deviceset="TP" device="TP15R"/>
+<part name="R1" library="resistor" deviceset="R-EU_" device="R0805" value="10K"/>
+<part name="+3V8" library="supply1" deviceset="+3V3" device=""/>
+<part name="J1" library="SparkFun-Connectors" deviceset="M03" device="1X03_NO_SILK"/>
+<part name="J2" library="SparkFun-Connectors" deviceset="M04" device="NO_SILK_ALL_ROUND"/>
 </parts>
 <sheets>
@@
 <instance part="C1" gate="G$1" x="68.58" y="142.24"/>
 <instance part="C2" gate="G$1" x="99.06" y="142.24"/>
-<instance part="P+1" gate="1" x="38.1" y="154.94" rot="R90"/>
+<instance part="P+1" gate="1" x="144.78" y="139.7"/>
 <instance part="P+3" gate="1" x="35.56" y="144.78"/>
 <instance part="GND1" gate="1" x="35.56" y="119.38"/>
-<instance part="GND3" gate="1" x="149.86" y="114.3"/>
-<instance part="GND4" gate="1" x="162.56" y="104.14"/>
-<instance part="GND5" gate="1" x="165.1" y="116.84"/>
-<instance part="GND6" gate="1" x="152.4" y="96.52"/>
+<instance part="GND3" gate="1" x="144.78" y="124.46"/>
+<instance part="GND6" gate="1" x="154.94" y="68.58"/>
 <instance part="U$2" gate="G$1" x="60.96" y="111.76" smashed="yes"/>
 <instance part="+3V1" gate="G$1" x="73.66" y="121.92"/>
-<instance part="+3V2" gate="G$1" x="111.76" y="121.92"/>
-<instance part="+3V3" gate="G$1" x="124.46" y="154.94" rot="R270"/>
-<instance part="+3V5" gate="G$1" x="127" y="147.32" rot="R270"/>
-<instance part="GND7" gate="1" x="25.4" y="104.14"/>
-<instance part="GND8" gate="1" x="20.32" y="96.52"/>
+<instance part="+3V3" gate="G$1" x="154.94" y="86.36"/>
 <instance part="GND9" gate="1" x="73.66" y="104.14"/>
-<instance part="GND10" gate="1" x="17.78" y="109.22"/>
 <instance part="R2" gate="G$1" x="45.72" y="96.52" rot="R90"/>
 <instance part="GND11" gate="1" x="45.72" y="88.9"/>
@@
 <attribute name="VALUE" x="117.602" y="82.55" size="1.778" layer="96" rot="R90"/>
 </instance>
+<instance part="R6" gate="G$1" x="127" y="114.3" smashed="yes" rot="R270">
+<attribute name="NAME" x="128.4986" y="115.57" size="1.778" layer="95" rot="R270"/>
+<attribute name="VALUE" x="123.698" y="115.57" size="1.778" layer="96" rot="R270"/>
+</instance>
+<instance part="+3V7" gate="G$1" x="127" y="124.46" smashed="yes">
+<attribute name="VALUE" x="124.46" y="119.38" size="1.778" layer="96" rot="R90"/>
+</instance>
+<instance part="TP1" gate="G$1" x="132.08" y="106.68" rot="R270"/>
+<instance part="R1" gate="G$1" x="111.76" y="121.92" smashed="yes" rot="R270">
+<attribute name="NAME" x="113.2586" y="123.19" size="1.778" layer="95" rot="R270"/>
+<attribute name="VALUE" x="108.458" y="123.19" size="1.778" layer="96" rot="R270"/>
+</instance>
+<instance part="+3V8" gate="G$1" x="111.76" y="132.08" smashed="yes">
+<attribute name="VALUE" x="109.22" y="127" size="1.778" layer="96" rot="R90"/>
+</instance>
+<instance part="J1" gate="J$1" x="154.94" y="132.08" rot="R180"/>
+<instance part="J2" gate="G$1" x="162.56" y="78.74" rot="R180"/>
 </instances>
 <busses>
@@
 <wire x1="35.56" y1="137.16" x2="35.56" y2="142.24" width="0.1524" layer="91"/>
 </segment>
+<segment>
+<pinref part="J1" gate="J$1" pin="1"/>
+<wire x1="147.32" y1="134.62" x2="144.78" y2="134.62" width="0.1524" layer="91"/>
+<pinref part="P+1" gate="1" pin="+5V"/>
+<wire x1="144.78" y1="134.62" x2="144.78" y2="137.16" width="0.1524" layer="91"/>
+</segment>
 </net>
 <net name="GND" class="0">
@@
 </segment>
 <segment>
+<pinref part="J1" gate="J$1" pin="3"/>
+<wire x1="147.32" y1="129.54" x2="144.78" y2="129.54" width="0.1524" layer="91"/>
+<pinref part="GND3" gate="1" pin="GND"/>
+<wire x1="144.78" y1="129.54" x2="144.78" y2="127" width="0.1524" layer="91"/>
+</segment>
+<segment>
+<pinref part="J2" gate="G$1" pin="4"/>
+<wire x1="157.48" y1="73.66" x2="154.94" y2="73.66" width="0.1524" layer="91"/>
+<pinref part="GND6" gate="1" pin="GND"/>
+<wire x1="154.94" y1="73.66" x2="154.94" y2="71.12" width="0.1524" layer="91"/>
+</segment>
+<segment>
 <pinref part="U$1" gate="G$1" pin="GND7"/>
+<wire x1="76.2" y1="109.22" x2="73.66" y2="109.22" width="0.1524" layer="91"/>
 <pinref part="GND9" gate="1" pin="GND"/>
-<wire x1="76.2" y1="109.22" x2="73.66" y2="109.22" width="0.1524" layer="91"/>
 <wire x1="73.66" y1="109.22" x2="73.66" y2="106.68" width="0.1524" layer="91"/>
 </segment>
@@
 </segment>
 <segment>
-<pinref part="U$1" gate="G$1" pin="CH_PD"/>
-<pinref part="+3V2" gate="G$1" pin="+3V3"/>
-<wire x1="109.22" y1="114.3" x2="111.76" y2="114.3" width="0.1524" layer="91"/>
-<wire x1="111.76" y1="114.3" x2="111.76" y2="119.38" width="0.1524" layer="91"/>
-</segment>
-<segment>
 <pinref part="LED2" gate="G$1" pin="A"/>
 <pinref part="+3V6" gate="G$1" pin="+3V3"/>
 <wire x1="45.72" y1="109.22" x2="45.72" y2="116.84" width="0.1524" layer="91"/>
+</segment>
+<segment>
+<pinref part="+3V7" gate="G$1" pin="+3V3"/>
+<pinref part="R6" gate="G$1" pin="1"/>
+<wire x1="127" y1="121.92" x2="127" y2="119.38" width="0.1524" layer="91"/>
+</segment>
+<segment>
+<pinref part="+3V8" gate="G$1" pin="+3V3"/>
+<pinref part="R1" gate="G$1" pin="1"/>
+<wire x1="111.76" y1="129.54" x2="111.76" y2="127" width="0.1524" layer="91"/>
+</segment>
+<segment>
+<pinref part="J2" gate="G$1" pin="1"/>
+<wire x1="157.48" y1="81.28" x2="154.94" y2="81.28" width="0.1524" layer="91"/>
+<pinref part="+3V3" gate="G$1" pin="+3V3"/>
+<wire x1="154.94" y1="81.28" x2="154.94" y2="83.82" width="0.1524" layer="91"/>
 </segment>
 </net>
@@
 </segment>
 </net>
+<net name="N$4" class="0">
+<segment>
+<pinref part="U$1" gate="G$1" pin="GPIO0"/>
+<wire x1="109.22" y1="106.68" x2="127" y2="106.68" width="0.1524" layer="91"/>
+<wire x1="127" y1="106.68" x2="127" y2="109.22" width="0.1524" layer="91"/>
+<pinref part="R6" gate="G$1" pin="2"/>
+<pinref part="TP1" gate="G$1" pin="TP"/>
+<wire x1="127" y1="106.68" x2="129.54" y2="106.68" width="0.1524" layer="91"/>
+<junction x="127" y="106.68"/>
+</segment>
+</net>
+<net name="N$5" class="0">
+<segment>
+<wire x1="111.76" y1="114.3" x2="111.76" y2="116.84" width="0.1524" layer="91"/>
+<pinref part="R1" gate="G$1" pin="2"/>
+<pinref part="U$1" gate="G$1" pin="CH_PD"/>
+<wire x1="109.22" y1="114.3" x2="111.76" y2="114.3" width="0.1524" layer="91"/>
+</segment>
+</net>
+<net name="RX" class="0">
+<segment>
+<pinref part="U$1" gate="G$1" pin="RX"/>
+<wire x1="109.22" y1="111.76" x2="111.76" y2="111.76" width="0.1524" layer="91"/>
+<label x="111.76" y="111.76" size="1.27" layer="95" xref="yes"/>
+</segment>
+<segment>
+<pinref part="J2" gate="G$1" pin="2"/>
+<wire x1="157.48" y1="78.74" x2="154.94" y2="78.74" width="0.1524" layer="91"/>
+<label x="154.94" y="78.74" size="1.27" layer="95" rot="MR0" xref="yes"/>
+</segment>
+</net>
+<net name="TX" class="0">
+<segment>
+<pinref part="U$1" gate="G$1" pin="TX"/>
+<wire x1="109.22" y1="109.22" x2="111.76" y2="109.22" width="0.1524" layer="91"/>
+<label x="111.76" y="109.22" size="1.27" layer="95" xref="yes"/>
+</segment>
+<segment>
+<pinref part="J2" gate="G$1" pin="3"/>
+<wire x1="157.48" y1="76.2" x2="154.94" y2="76.2" width="0.1524" layer="91"/>
+<label x="154.94" y="76.2" size="1.27" layer="95" rot="MR0" xref="yes"/>
+</segment>
+</net>
+<net name="SIG_PIXEL" class="0">
+<segment>
+<pinref part="U$1" gate="G$1" pin="GPIO2"/>
+<wire x1="109.22" y1="104.14" x2="111.76" y2="104.14" width="0.1524" layer="91"/>
+<label x="111.76" y="104.14" size="1.27" layer="95" xref="yes"/>
+</segment>
+<segment>
+<pinref part="J1" gate="J$1" pin="2"/>
+<wire x1="147.32" y1="132.08" x2="144.78" y2="132.08" width="0.1524" layer="91"/>
+<label x="144.78" y="132.08" size="1.27" layer="95" rot="MR0" xref="yes"/>
+</segment>
+</net>
